File: SigGen.kicad_pcb (KiCad board)
At the start: 2 copper layers, 37 parts, among them IC1 ATTINY2313-P, IC2 ATTINY2313-P, P1 USB_A, P2 CONN_01X05, U2 4N25, U3 DCDC_5V/5V, Y1 12MHz, Y2 20MHz

Commit message: Finished the PCB
Parts:
- removed JP1: JUMPER, Socket_Strips:Socket_Strip_Straight_1x03
- removed U3: DCDC_5V/5V, Socket_Strips:Socket_Strip_Straight_1x04
- added C8: 10u, Capacitors_SMD:C_0805_HandSoldering, F.Cu at (99.1, 86.4)
- added P3: CONN_01X03, Socket_Strips:Socket_Strip_Straight_1x03, F.Cu at (110.5, 92.7)
- added U1: DCDC_convertor, Socket_Strips:Socket_Strip_Straight_1x04, F.Cu at (105.4, 85.1)
- moved P2 43.6 mm to (136.7, 95.2)
- moved C1 43.6 mm to (126.5, 94.0), turned to 90 degrees
- moved R8 32.6 mm to (139.2, 93.7)
- moved D2 29.3 mm to (106.7, 97.8), turned to 180 degrees
- moved D3 25.4 mm to (111.8, 97.8), turned to 180 degrees
- moved D4 18.5 mm to (111.8, 95.2)
- moved D1 17.1 mm to (105.4, 94.0), turned to 90 degrees
- moved R2 15.7 mm to (114.3, 90.2)
- moved C5 15.0 mm to (141.5, 93.7), turned to 270 degrees
- moved Y2 13.0 mm to (115.6, 97.8)
- moved C4 12.8 mm to (102.9, 86.4), turned to 90 degrees
- moved R17 11.9 mm to (125.2, 87.6)
- moved C6 11.9 mm to (124.0, 95.2)
- moved C7 11.9 mm to (124.0, 97.8)
- moved IC1 11.9 mm to (121.4, 87.6)
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Connections:
- IC1 pad 11: (no net) -> Net-(IC1-Pad11)
- IC1 pad 3: (no net) -> Net-(IC1-Pad3)
- IC1 pad 6: (no net) -> Net-(IC1-Pad6)
- IC1 pad 7: (no net) -> Net-(IC1-Pad7)
- IC1 pad 8: (no net) -> Net-(IC1-Pad8)
- IC1 pad 9: (no net) -> Net-(IC1-Pad9)
- IC2 pad 11: (no net) -> Net-(IC2-Pad11)
- IC2 pad 12: (no net) -> Net-(IC2-Pad12)
- IC2 pad 13: (no net) -> Net-(IC2-Pad13)
- IC2 pad 14: (no net) -> Net-(IC2-Pad14)
- IC2 pad 15: (no net) -> Net-(IC2-Pad15)
- IC2 pad 16: (no net) -> Net-(IC2-Pad16)
- IC2 pad 17: (no net) -> Net-(IC2-Pad17)
- IC2 pad 18: (no net) -> Net-(IC2-Pad18)
- IC2 pad 19: (no net) -> Net-(IC2-Pad19)
- IC2 pad 2: (no net) -> Net-(IC2-Pad2)
- IC2 pad 8: (no net) -> Net-(IC2-Pad8)
- IC2 pad 9: (no net) -> Net-(IC2-Pad9)
- R3 pad 1: Net-(R3-Pad1) -> Net-(IC2-Pad3)
- R3 pad 2: Net-(C4-Pad1) -> Net-(R3-Pad2)
- R4 pad 1: Net-(C4-Pad1) -> Net-(IC2-Pad8)
- U2 pad 1: Net-(R3-Pad1) -> Net-(R3-Pad2)
- U2 pad 2: Net-(IC2-Pad3) -> Net-(IC2-Pad12)
- U2 pad 6: (no net) -> Net-(U2-Pad6)
Routing:
- net Net-(C1-Pad1): track 0.00 -> 101.5 mm
- net Net-(C2-Pad2): track 0.00 -> 86.5 mm
- net Net-(C4-Pad1): track 0.00 -> 55.1 mm, vias 0 -> 2
- net Net-(C1-Pad2): track 0.00 -> 43.9 mm
- net Net-(IC1-Pad2): track 0.00 -> 43.1 mm, vias 0 -> 2
- net Net-(D1-Pad2): track 0.00 -> 38.9 mm
- net Net-(R3-Pad2): track 0.00 -> 20.2 mm
- net Net-(P2-Pad2): track 0.00 -> 20.2 mm
- net Net-(C2-Pad1): track 0.00 -> 10.9 mm
- net Net-(C7-Pad1): track 0.00 -> 9.57 mm
- net Net-(P1-Pad2): track 0.00 -> 8.06 mm
- net Net-(IC2-Pad8): track 0.00 -> 7.76 mm
- net Net-(C3-Pad1): track 0.00 -> 7.72 mm
- net Net-(P1-Pad3): track 0.00 -> 7.59 mm
- net Net-(C6-Pad1): track 0.00 -> 7.31 mm
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
Commit message: Updated SCHEMATIC
Connections:
- IC1 pad 11: Net-(IC1-Pad11) -> (no net)
- IC1 pad 3: Net-(IC1-Pad3) -> (no net)
- IC1 pad 6: Net-(IC1-Pad6) -> (no net)
- IC1 pad 7: Net-(IC1-Pad7) -> (no net)
- IC1 pad 8: Net-(IC1-Pad8) -> (no net)
- IC1 pad 9: Net-(IC1-Pad9) -> (no net)
- IC2 pad 11: Net-(IC2-Pad11) -> (no net)
- IC2 pad 12: Net-(IC2-Pad12) -> (no net)
- IC2 pad 13: Net-(IC2-Pad13) -> (no net)
- IC2 pad 14: Net-(IC2-Pad14) -> (no net)
- IC2 pad 15: Net-(IC2-Pad15) -> (no net)
- IC2 pad 16: Net-(IC2-Pad16) -> (no net)
- IC2 pad 17: Net-(IC2-Pad17) -> (no net)
- IC2 pad 18: Net-(IC2-Pad18) -> (no net)
- IC2 pad 19: Net-(IC2-Pad19) -> (no net)
- IC2 pad 2: Net-(IC2-Pad2) -> (no net)
- IC2 pad 9: Net-(IC2-Pad9) -> (no net)
- U2 pad 1: Net-(R3-Pad2) -> Net-(C4-Pad1)
- U2 pad 2: Net-(IC2-Pad12) -> Net-(R3-Pad2)
- U2 pad 6: Net-(U2-Pad6) -> (no net)
Routing:
- net Net-(C4-Pad1): track 55.1 -> 75.4 mm
- net Net-(IC2-Pad12): track 2.54 -> 0.00 mm
- net Net-(R3-Pad2): track 20.2 -> 22.0 mm
