File: SigGen.sch (KiCad schematic (older format))
At the start: 19 parts, among them IC1 ATTINY2313-P, U1 4N25, U2 4N25, U3 DCDC_5V/5V

Commit message: Updated schematic
Parts:
- removed R1: R, symbol R
- removed R4: 2K2, symbol R
- removed U1: 4N25, DIP-6, symbol 4N25
- added C?: 4u7, symbol C
- added C? (x2): 22p, symbol C
- added D? (x4): D, symbol D
- added JP?: JUMPER, symbol JUMPER
- added P?: CONN_01X05, symbol CONN_01X05
- added R?: 10K, symbol R
- added R? (x10): 220R, symbol R
- added Y?: 20MHz, symbol Crystal
- C?: value C -> 4u7
- R2: value R -> 2K2
- R3: value R -> 220R
- Y?: value Crystal -> 12MHz
Connections:
- net at IC1.1 (PA2(~RESET~/dW)): now also R?.1
- net at IC1.12 ((PCINT0/AIN0)PB0): now also R?.1
- net at IC1.13 ((PCINT1/AIN1)PB1): now also R?.1
- net at IC1.14 ((PCINT2/OC0A)PB2): now also R?.1
- net at IC1.15 ((PCINT3/OC1A)PB3): now also R?.1
- net at IC1.16 ((PCINT4/OC1B)PB4): now also R?.1
- net at IC1.17 ((PCINT5/MOSI/DI/SDA)PB5): now also R?.1
- net at IC1.18 ((PCINT6/MISO/DO)PB6): now also R?.1
- net at IC1.19 ((PCINT7/USCK/SCK/SCL)PB7): now also R?.1
- net at IC1.4 (PA1(XTAL2)): now also C?.1, Y?.1
- net at IC1.5 (PA0(XTAL1)): now also C?.1, Y?.2
- net at C?.2, C?.2, IC?.10 (GND)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: now also C?.2; no longer C?.1, U2.2
- net at IC?.20 (VCC), P?.1 (VCC), R?.1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: now also C?.1, R3.2, R?.2; no longer C?.2, R?.1
- net at U2.1: now also R3.1; no longer R3.2
- net at IC?.3 ((TXD)PD1): now also U2.2; no longer R3.1
- net at IC?.1 (PA2(~RESET~/dW)): now also R?.1; no longer R?.2
- net GNDREF: no longer names the net of IC1.10 (GND), U3.3 (out-)
- net GNDREF: now also C1.1, U2.4, C?.2, C?.2, C?.2, P?.1 (P1), R?.2; no longer C1.2, R2.2
- new net: IC1.2 ((RXD)PD0), R2.2, U2.5
- new net: C1.2, D?.1 (K), IC1.20 (VCC), JP?.2, P?.4 (P4), R2.1, R?.1, R?.2
- new net: D?.2 (A), JP?.1, P?.5 (P5), U3.4 (out+)
- new net: D?.1 (K), D?.2 (A) (x3)
- new net: P?.2 (P2), R?.2, R?.2, R?.2, R?.2, R?.2, R?.2, R?.2, R?.2
- new net: C?.1, P?.3 (P3), R?.1, R?.2
- no-connect marks 2 -> 19
Other:
- note added: "+5V"
- note added: "GND"
- note added: "Vdd"
- note added: "Vdd/2"
- note added: "sig"
- moved on the sheet: C1, C?, IC1, IC?, P?, R2, R3, R?, U2, U3, Y?

Commit message: Updating PCB
Parts:
- C1: value C -> 100n; footprint (none) -> Capacitors_SMD:C_0805_HandSoldering
- C2, C3, C4, C5, C6, C7: renamed from C?; footprint (none) -> Capacitors_SMD:C_0805_HandSoldering
- D1, D2, D3, D4: renamed from D?; footprint (none) -> Capacitors_SMD:C_0805_HandSoldering
- IC1: footprint DIP20 -> Housings_DIP:DIP-20_W7.62mm
- IC2: renamed from IC?; footprint DIP20 -> Housings_DIP:DIP-20_W7.62mm
- JP1: renamed from JP?; footprint (none) -> Socket_Strips:Socket_Strip_Straight_1x03
- P1: renamed from P?; footprint (none) -> Connect:USB_A
- P2: renamed from P?; footprint (none) -> Socket_Strips:Socket_Strip_Straight_1x05
- R1, R10, R11, R12, R13, R14, R15, R16, R17, R4, R5, R6, R7, R8, R9: renamed from R?; footprint (none) -> Resistors_SMD:R_0805_HandSoldering
- R2, R3: footprint (none) -> Resistors_SMD:R_0805_HandSoldering
- U2: footprint DIP-6 -> Housings_DIP:DIP-6_W7.62mm
- U3: footprint (none) -> Socket_Strips:Socket_Strip_Straight_1x04
- Y1, Y2: renamed from Y?; footprint (none) -> Crystals:Crystal_HC49-U_Vertical

Commit message: Finished the PCB
Parts:
- removed JP1: JUMPER, Socket_Strips:Socket_Strip_Straight_1x03, symbol JUMPER
- removed U3: DCDC_5V/5V, Socket_Strips:Socket_Strip_Straight_1x04, symbol DCDC_convertor
- added C8: 10u, Capacitors_SMD:C_0805_HandSoldering, symbol C
- added P3: CONN_01X03, Socket_Strips:Socket_Strip_Straight_1x03, symbol CONN_01X03
- added U1: DCDC_convertor, Socket_Strips:Socket_Strip_Straight_1x04, symbol DCDC_convertor
Connections:
- net at C1.1, C5.2, C6.2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: now also U1.3 (out-)
- net at C1.2, D4.1 (K), IC1.20 (VCC)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: now also P3.1 (P1), P3.2 (P2)
- net at C2.2, C3.2, C4.2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: now also C8.2, U1.1 (in-)
- net at C4.1, IC2.20 (VCC), P1.1 (VCC)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: now also C8.1, U1.2 (in+); no longer R3.2, R4.1
- net at D1.2 (A), P2.5 (P5): now also P3.3 (P3), U1.4 (out+)
- net at U2.1: now also R3.2; no longer R3.1
- net at U2.2: now also IC2.12 ((PCINT0/AIN0)PB0); no longer IC2.3 ((TXD)PD1)
- net at IC2.8 ((T0)PD4): now also R4.1
- new net: IC2.3 ((TXD)PD1), R3.1
- no-connect marks 19 -> 17
Other:
- moved on the sheet: R3
Changed lines of the file:
@@
-$EndComp
-$Comp
-L DCDC_convertor U3
-U 1 1 5831CFB3
-P 5450 2700
-F 0 "U3" H 5850 3100 60  0000 C CNN
-F 1 "DCDC_5V/5V" H 5300 3100 60  0000 C CNN
-F 2 "Socket_Strips:Socket_Strip_Straight_1x04" H 5450 2700 60  0001 C CNN
-F 3 "" H 5450 2700 60  0001 C CNN
-	1    5450 2700
-	1    0    0    -1
 $EndComp
 $Comp
@@
 L R R3
 U 1 1 5831DE1F
-P 4650 3950
-F 0 "R3" V 4730 3950 50  0000 C CNN
-F 1 "220R" V 4650 3950 50  0000 C CNN
-F 2 "Resistors_SMD:R_0805_HandSoldering" V 4580 3950 50  0001 C CNN
-F 3 "" H 4650 3950 50  0000 C CNN
-	1    4650 3950
-	1    0    0    1
+P 4700 4450
+F 0 "R3" V 4780 4450 50  0000 C CNN
+F 1 "220R" V 4700 4450 50  0000 C CNN
+F 2 "Resistors_SMD:R_0805_HandSoldering" V 4630 4450 50  0001 C CNN
+F 3 "" H 4700 4450 50  0000 C CNN
+	1    4700 4450
+	0    -1   1    0
 $EndComp
 $Comp
@@
 	1900 5950 1900 6400
 Wire Wire Line
-	1150 6000 2100 6000
-Wire Wire Line
 	2100 6000 2100 6100
 Wire Wire Line
@@
 $EndComp
 $Comp
-L JUMPER JP1
-U 1 1 58335221
-P 7000 2100
-F 0 "JP1" H 7000 2250 50  0000 C CNN
-F 1 "JUMPER" H 7000 2020 50  0000 C CNN
-F 2 "Socket_Strips:Socket_Strip_Straight_1x03" H 7000 2100 50  0001 C CNN
-F 3 "" H 7000 2100 50  0000 C CNN
-	1    7000 2100
-	1    0    0    -1
-$EndComp
-$Comp
 L D D1
 U 1 1 58335391
@@
 	7150 2550 7200 2550
 Wire Wire Line
-	6100 2100 6700 2100
-Wire Wire Line
-	7300 2100 8900 2100
+	6100 2100 6850 2100
+Wire Wire Line
+	6950 2100 8900 2100
 Wire Wire Line
 	2000 3900 2000 3750
@@
 Wire Wire Line
 	1300 2850 1300 5600
-Wire Wire Line
-	1300 5600 3300 5600
 Connection ~ 3300 5600
 Connection ~ 1900 5600
 Wire Wire Line
 	1900 5650 1900 5600
-Wire Wire Line
-	4450 4450 5150 4450
-Wire Wire Line
-	4650 4250 4650 4100
-Wire Wire Line
-	4650 3800 4650 2550
-Connection ~ 4650 2550
-Wire Wire Line
-	4650 4250 5150 4250
 NoConn ~ 5750 4250
 Wire Wire Line
@@
 Connection ~ 8900 5400
 Connection ~ 10750 4350
-NoConn ~ 4450 3450
-NoConn ~ 4450 3550
-NoConn ~ 4450 3650
 NoConn ~ 4450 3750
 NoConn ~ 4450 3850
@@
 NoConn ~ 4450 4150
 NoConn ~ 4450 4350
-NoConn ~ 4450 4750
 NoConn ~ 4450 4850
 NoConn ~ 4450 4950
@@
 Text Notes 7050 6300 1    60   ~ 0
 GND
+$Comp
+L DCDC_convertor U1
+U 1 1 5836E6F0
+P 5450 2700
+F 0 "U1" H 6000 3400 60  0000 C CNN
+F 1 "DCDC_convertor" H 5450 3400 60  0000 C CNN
+F 2 "Socket_Strips:Socket_Strip_Straight_1x04" H 5450 2700 60  0001 C CNN
+F 3 "" H 5450 2700 60  0001 C CNN
+	1    5450 2700
+	1    0    0    -1
+$EndComp
+Wire Wire Line
+	1150 6000 1900 6000
+Wire Wire Line
+	2100 6000 4600 6000
+Wire Wire Line
+	4600 6000 4600 4750
+Wire Wire Line
+	4600 4750 4450 4750
+Wire Wire Line
+	4450 4450 4550 4450
+Wire Wire Line
+	4850 4450 4850 4250
+Wire Wire Line
+	4850 4250 5150 4250
+Wire Wire Line
+	5050 4450 5150 4450
+Wire Wire Line
+	5050 3450 5050 4450
+NoConn ~ 4450 3650
+NoConn ~ 4450 3550
+Wire Wire Line
+	4450 3450 5050 3450
+$Comp
+L CONN_01X03 P3
+U 1 1 58370475
+P 6950 1800
+F 0 "P3" H 6950 2000 50  0000 C CNN
+F 1 "CONN_01X03" V 7050 1800 50  0000 C CNN
+F 2 "Socket_Strips:Socket_Strip_Straight_1x03" H 6950 1800 50  0001 C CNN
+F 3 "" H 6950 1800 50  0000 C CNN
+	1    6950 1800
+	0    1    -1   0
+$EndComp
+Wire Wire Line
+	6850 2100 6850 2000
+Wire Wire Line
+	6950 2100 6950 2000
+Wire Wire Line
+	7050 2000 7050 2100
+Connection ~ 7050 2100
+Wire Wire Line
+	1300 5600 3300 5600
+$Comp
+L C C8
+U 1 1 58370690
+P 4600 2700
+F 0 "C8" H 4625 2800 50  0000 L CNN
+F 1 "10u" H 4625 2600 50  0000 L CNN
+F 2 "Capacitors_SMD:C_0805_HandSoldering" H 4638 2550 50  0001 C CNN
+F 3 "" H 4600 2700 50  0000 C CNN
+	1    4600 2700
+	-1   0    0    -1
+$EndComp
+Connection ~ 4600 2550
+Connection ~ 4600 2850
 $EndSCHEMATC

Commit message: Updated SCHEMATIC
Connections:
- net at U2.1: now also C4.1, C8.1, IC2.20 (VCC), P1.1 (VCC), R1.2, U1.2 (in+); no longer R3.2
- net at U2.2: now also R3.2; no longer IC2.12 ((PCINT0/AIN0)PB0)
- no-connect marks 17 -> 18
Changed lines of the file:
@@
 Wire Wire Line
 	4450 4450 4550 4450
-Wire Wire Line
-	4850 4450 4850 4250
-Wire Wire Line
-	4850 4250 5150 4250
-Wire Wire Line
-	5050 4450 5150 4450
-Wire Wire Line
-	5050 3450 5050 4450
 NoConn ~ 4450 3650
 NoConn ~ 4450 3550
-Wire Wire Line
-	4450 3450 5050 3450
 $Comp
 L CONN_01X03 P3
@@
 Connection ~ 4600 2550
 Connection ~ 4600 2850
+Wire Wire Line
+	5050 3100 5050 4250
+Wire Wire Line
+	5050 4250 5150 4250
+Wire Wire Line
+	4850 4450 5150 4450
+Wire Wire Line
+	5050 3100 3300 3100
+Connection ~ 3300 3100
+NoConn ~ 4450 3450
 $EndSCHEMATC
